Commit message: Start joint state publisher gui along with rviz Move base link from the center of the base cylinder   to its base

File: urdf/my_rb1.xacro (robot description, xacro)
@@ -50,4 +50,5 @@
             <parent link="base_link"/>
             <child link="base_cylinder_link"/>
+            <origin rpy="0.0 0 0" xyz="0 0 ${base_cylinder_height * 0.5}"/>
         </joint>
     </xacro:macro>

Commit message: rb1 base cylinder is dark blue in rviz

File: urdf/my_rb1.xacro (robot description, xacro)
@@ -11,6 +11,6 @@
     <xacro:property name="base_cylinder_mass" value="25"/>
     <xacro:macro name="rviz_materials">
-        <material name="grey">
-            <color rgba="0.75 0.75 0.75 1"/>
+        <material name="dark_blue">
+            <color rgba="0 0 0.55 1"/>
         </material>
     </xacro:macro>
@@ -39,4 +39,5 @@
                     <cylinder radius="${base_cylinder_radius}" length="${base_cylinder_height}"/>
                 </geometry>
+                <material name="dark_blue"/>
             </visual>
         </link>

Commit message: Fix rviz color dark blue

File: urdf/my_rb1.xacro (robot description, xacro)
@@ -10,9 +10,7 @@
     <xacro:property name="base_cylinder_height" value="0.3"/>
     <xacro:property name="base_cylinder_mass" value="25"/>
-    <xacro:macro name="rviz_materials">
-        <material name="dark_blue">
-            <color rgba="0 0 0.55 1"/>
-        </material>
-    </xacro:macro>
+    <material name="dark_blue">
+        <color rgba="0 0 0.55 1"/>
+    </material>
     <!-- base cylinder XACRO -->
     <xacro:macro name="base_cylinder">

Commit message: Add wheels

File: urdf/my_rb1.xacro (robot description, xacro)
@@ -1,4 +1,8 @@
 <?xml version="1.0"?>
 <robot xmlns:xacro="http://www.ros.org/wiki/xacro" name="my_rb1">
+    <!-- All 4 wheels have the same mass -->
+    <xacro:property name="wheel_mass" value="0.25"/>
+    <xacro:property name="wheel_count" value="4"/>
+    <xacro:property name="base_cylinder_mass" value="${25 - (wheel_count*wheel_mass)}"/>
     <!-- Properties -->
     <xacro:property name="base_cylinder_kp" value="1000.0"/>
@@ -6,10 +10,26 @@
 	<xacro:property name="base_cylinder_mu1" value="10.0"/>
     <xacro:property name="base_cylinder_mu2" value="10.0"/>
+    <xacro:property name="wheel_kp" value="1000.0"/>
+	<xacro:property name="wheel_kd" value="1000.0"/>
+	<xacro:property name="wheel_mu1" value="10.0"/>
+    <xacro:property name="wheel_mu2" value="10.0"/>
     <!-- The robot is a cylinder 50 cm in diameter and 30 cm in height -->
     <xacro:property name="base_cylinder_radius" value="0.25"/>
     <xacro:property name="base_cylinder_height" value="0.3"/>
-    <xacro:property name="base_cylinder_mass" value="25"/>
+    <!-- Has 2 wheels of 5 cm diameter on each side of the base. One at (0.1, -0.2, -0.15)
+         from the base_link and another at (0.1, 0.2, -0.15). -->
+    <xacro:property name="wheel_radius" value="0.025"/>
+    <xacro:property name="wheel_height" value="0.025"/>
+    <xacro:property name="wheel_x" value="0.1"/>
+    <xacro:property name="left_wheel_y" value="-0.2"/>
+    <xacro:property name="wheel_z" value="-0.15"/>
+    <xacro:property name="wheel_roll" value="1.57"/>
+    <xacro:property name="wheel_pitch" value="0"/>
+    <xacro:property name="wheel_yaw" value="0"/>
     <material name="dark_blue">
         <color rgba="0 0 0.55 1"/>
+    </material>
+    <material name="black">
+        <color rgba="0 0 0 1"/>
     </material>
     <!-- base cylinder XACRO -->
@@ -46,8 +66,48 @@
             <kd>${base_cylinder_kd}</kd>
         </gazebo>
-        <joint name="fixed" type="fixed">
+        <joint name="base_cylinder_base_link_joint" type="fixed">
             <parent link="base_link"/>
             <child link="base_cylinder_link"/>
-            <origin rpy="0.0 0 0" xyz="0 0 ${base_cylinder_height * 0.5}"/>
+            <!--<origin rpy="0.0 0 0" xyz="0 0 ${base_cylinder_height * 0.5}"/>-->
+            <origin rpy="0.0 0 0" xyz="0 0 0"/>
+        </joint>
+    </xacro:macro>
+    <xacro:macro name="wheel" params="side">
+        <xacro:property name="multiplier" value="${-1 if side == 'right' else 1}"/>
+        <xacro:property name="current_wheel_name" value="${side}_wheel_link"/>
+        <link name="${current_wheel_name}">
+            <inertial>
+                <origin xyz="0 0 0" rpy="0 0 0"/>
+                <mass value="${wheel_mass}" />
+                <xacro:cylinder_inertia mass="${wheel_mass}"
+                    r="${wheel_radius}"
+                    l="${wheel_height}"
+                />
+            </inertial>
+            <collision>
+                <origin xyz="0 0 0" rpy="0 0 0"/>
+                <geometry>
+                    <cylinder radius="${wheel_radius}" length="${wheel_height}"/>
+                </geometry>
+            </collision>
+            <visual>
+                <origin rpy="0 0 0" xyz="0 0 0"/>
+                <geometry>
+                    <cylinder radius="${wheel_radius}" length="${wheel_height}"/>
+                </geometry>
+                <material name="black"/>
+            </visual>
+        </link>
+        <gazebo reference="${current_wheel_name}">
+            <mu1>${wheel_mu1}</mu1>
+            <mu2>${wheel_mu2}</mu2>
+            <kp>${wheel_kp}</kp>
+            <kd>${wheel_kd}</kd>
+        </gazebo>
+        <joint name="${current_wheel_name}_base_link_joint" type="continuous">
+            <parent link="base_link"/>
+            <child link="${current_wheel_name}"/>
+            <origin xyz="${wheel_x} ${multiplier * left_wheel_y} ${wheel_z}" rpy="${wheel_roll} ${wheel_pitch} ${wheel_yaw}" />
+             <axis xyz="0 0 1"/>
         </joint>
     </xacro:macro>
@@ -72,3 +132,5 @@
     </xacro:macro>
     <xacro:base_cylinder />
+    <xacro:wheel side="left" />
+    <xacro:wheel side="right" />
 </robot>

Commit message: Add casters

File: urdf/my_rb1.xacro (robot description, xacro)
@@ -3,6 +3,10 @@
     <!-- All 4 wheels have the same mass -->
     <xacro:property name="wheel_mass" value="0.25"/>
-    <xacro:property name="wheel_count" value="4"/>
-    <xacro:property name="base_cylinder_mass" value="${25 - (wheel_count*wheel_mass)}"/>
+    <xacro:property name="caster_mass" value="${wheel_mass}"/>
+    <xacro:property name="wheel_count" value="2"/>
+    <xacro:property name="wheel_mass_total" value="${wheel_count * wheel_mass}"/>
+    <xacro:property name="caster_count" value="2"/>
+    <xacro:property name="caster_mass_total" value="${caster_count * caster_mass}"/>
+    <xacro:property name="base_cylinder_mass" value="${25 - (wheel_mass_total + caster_mass_total)}"/>
     <!-- Properties -->
     <xacro:property name="base_cylinder_kp" value="1000.0"/>
@@ -14,4 +18,8 @@
 	<xacro:property name="wheel_mu1" value="10.0"/>
     <xacro:property name="wheel_mu2" value="10.0"/>
+    <xacro:property name="caster_kp" value="1000.0"/>
+	<xacro:property name="caster_kd" value="1000.0"/>
+	<xacro:property name="caster_mu1" value="0"/>
+    <xacro:property name="caster_mu2" value="0"/>
     <!-- The robot is a cylinder 50 cm in diameter and 30 cm in height -->
     <xacro:property name="base_cylinder_radius" value="0.25"/>
@@ -27,4 +35,11 @@
     <xacro:property name="wheel_pitch" value="0"/>
     <xacro:property name="wheel_yaw" value="0"/>
+    <!-- Has two caster wheels: one at the front and another at the back of the robot of 2.5 cm radius.
+         The friction parameters must be "0". One at (-0.1, 0.0, -0.15) from the base_link and another
+         at (0.1, 0.0, -0.15).-->
+    <xacro:property name="caster_radius" value="0.025"/>
+    <xacro:property name="front_caster_x" value="0.1"/>
+    <xacro:property name="caster_y" value="0"/>
+    <xacro:property name="caster_z" value="-0.15"/>
     <material name="dark_blue">
         <color rgba="0 0 0.55 1"/>
@@ -32,4 +47,7 @@
     <material name="black">
         <color rgba="0 0 0 1"/>
+    </material>
+    <material name="white">
+        <color rgba="1 1 1 1"/>
     </material>
     <!-- base cylinder XACRO -->
@@ -112,4 +130,43 @@
         </joint>
     </xacro:macro>
+    <xacro:macro name="caster" params="side">
+        <xacro:property name="multiplier" value="${-1 if side == 'front' else 1}"/>
+        <xacro:property name="current_caster_name" value="${side}_caster_link"/>
+        <link name="${current_caster_name}">
+            <inertial>
+                <origin xyz="0 0 0" rpy="0 0 0"/>
+                <mass value="${caster_mass}" />
+                <xacro:sphere_inertia mass="${caster_mass}"
+                    r="${caster_radius}"
+                />
+            </inertial>
+            <collision>
+                <origin xyz="0 0 0" rpy="0 0 0"/>
+                <geometry>
+                    <sphere radius="${caster_radius}"/>
+                </geometry>
+            </collision>
+            <visual>
+                <origin rpy="0 0 0" xyz="0 0 0"/>
+                <geometry>
+                    <sphere radius="${caster_radius}"/>
+                </geometry>
+                <material name="white"/>
+            </visual>
+        </link>
+        <gazebo reference="${current_caster_name}">
+            <mu1>${caster_mu1}</mu1>
+            <mu2>${caster_mu2}</mu2>
+            <kp>${caster_kp}</kp>
+            <kd>${caster_kd}</kd>
+        </gazebo>
+        <joint name="${current_caster_name}_base_link_joint" type="fixed">
+            <parent link="base_link"/>
+            <child link="${current_caster_name}"/>
+            <origin
+                xyz="${multiplier * front_caster_x} ${caster_y}  ${caster_z}"
+                rpy="0 0 0" />
+        </joint>
+    </xacro:macro>
     <!-- Math Usefull MACROS-->
     <xacro:macro  name="cylinder_inertia" params="mass r l">
@@ -134,3 +191,5 @@
     <xacro:wheel side="left" />
     <xacro:wheel side="right" />
+    <xacro:caster side="front" />
+    <xacro:caster side="back" />
 </robot>

Commit message: Add base_footprint

File: urdf/my_rb1.xacro (robot description, xacro)
@@ -55,4 +55,6 @@
         <link name="base_link">
         </link>
+        <link name="base_footprint">
+        </link>
         <link name="base_cylinder_link">
             <inertial>
@@ -87,6 +89,10 @@
             <parent link="base_link"/>
             <child link="base_cylinder_link"/>
-            <!--<origin rpy="0.0 0 0" xyz="0 0 ${base_cylinder_height * 0.5}"/>-->
             <origin rpy="0.0 0 0" xyz="0 0 0"/>
+        </joint>
+        <joint name="base_footprint_base_link_joint" type="fixed">
+            <parent link="base_link"/>
+            <child link="base_footprint"/>
+            <origin rpy="0.0 0 0" xyz="0 0 ${base_cylinder_height * -0.5}"/>
         </joint>
     </xacro:macro>

Commit message: Add front_laser link

File: urdf/my_rb1.xacro (robot description, xacro)
@@ -1,4 +1,14 @@
 <?xml version="1.0"?>
 <robot xmlns:xacro="http://www.ros.org/wiki/xacro" name="my_rb1">
+    <!--
+    'front_laser' link must be located at (0.25, 0.0, 0.075) from the 'base_link'.
+    Also the link must be rotated 180º in the `x` axis, this means, the laser is upside-down.
+    -->
+    <xacro:property name="front_laser_x" value="0.25"/>
+    <xacro:property name="front_laser_y" value="0.0"/>
+    <xacro:property name="front_laser_z" value="0.075"/>
+    <xacro:property name="front_laser_roll" value="3.14"/>
+    <xacro:property name="front_laser_pitch" value="0"/>
+    <xacro:property name="front_laser_yaw" value="0"/>
     <!-- All 4 wheels have the same mass -->
     <xacro:property name="wheel_mass" value="0.25"/>
@@ -57,4 +67,6 @@
         <link name="base_footprint">
         </link>
+        <link name="front_laser">
+        </link>
         <link name="base_cylinder_link">
             <inertial>
@@ -95,4 +107,11 @@
             <child link="base_footprint"/>
             <origin rpy="0.0 0 0" xyz="0 0 ${base_cylinder_height * -0.5}"/>
+        </joint>
+        <joint name="front_laser_base_link_joint" type="fixed">
+            <parent link="base_link"/>
+            <child link="front_laser"/>
+            <origin
+                xyz="${front_laser_x} ${front_laser_y} ${front_laser_z}"
+                rpy="${front_laser_roll} ${front_laser_pitch} ${front_laser_yaw}"/>
         </joint>
     </xacro:macro>

Commit message: Remove all kp and kd values because I don't understand them, and they just made rb1 fall through the floor. So only the frictionless caster values remain (mu1, mu2 = 0)

File: urdf/my_rb1.xacro (robot description, xacro)
@@ -20,14 +20,4 @@
     <xacro:property name="base_cylinder_mass" value="${25 - (wheel_mass_total + caster_mass_total)}"/>
     <!-- Properties -->
-    <xacro:property name="base_cylinder_kp" value="1000.0"/>
-	<xacro:property name="base_cylinder_kd" value="1000.0"/>
-	<xacro:property name="base_cylinder_mu1" value="10.0"/>
-    <xacro:property name="base_cylinder_mu2" value="10.0"/>
-    <xacro:property name="wheel_kp" value="1000.0"/>
-	<xacro:property name="wheel_kd" value="1000.0"/>
-	<xacro:property name="wheel_mu1" value="10.0"/>
-    <xacro:property name="wheel_mu2" value="10.0"/>
-    <xacro:property name="caster_kp" value="1000.0"/>
-	<xacro:property name="caster_kd" value="1000.0"/>
 	<xacro:property name="caster_mu1" value="0"/>
     <xacro:property name="caster_mu2" value="0"/>
@@ -93,8 +83,5 @@
         </link>
         <gazebo reference="base_cylinder_link">
-            <mu1>${base_cylinder_mu1}</mu1>
-            <mu2>${base_cylinder_mu2}</mu2>
-            <kp>${base_cylinder_kp}</kp>
-            <kd>${base_cylinder_kd}</kd>
+            <material>Gazebo/Blue</material>
         </gazebo>
         <joint name="base_cylinder_base_link_joint" type="fixed">
@@ -143,8 +130,5 @@
         </link>
         <gazebo reference="${current_wheel_name}">
-            <mu1>${wheel_mu1}</mu1>
-            <mu2>${wheel_mu2}</mu2>
-            <kp>${wheel_kp}</kp>
-            <kd>${wheel_kd}</kd>
+            <material>Gazebo/Black</material>
         </gazebo>
         <joint name="${current_wheel_name}_base_link_joint" type="continuous">
@@ -183,6 +167,5 @@
             <mu1>${caster_mu1}</mu1>
             <mu2>${caster_mu2}</mu2>
-            <kp>${caster_kp}</kp>
-            <kd>${caster_kd}</kd>
+            <material>Gazebo/White</material>
         </gazebo>
         <joint name="${current_caster_name}_base_link_joint" type="fixed">

Commit message: Fix sliding robot with better friction and contact   stiffness settings

File: urdf/my_rb1.xacro (robot description, xacro)
@@ -22,4 +22,8 @@
 	<xacro:property name="caster_mu1" value="0"/>
     <xacro:property name="caster_mu2" value="0"/>
+    <xacro:property name="wheel_kp" value="1000000.0"/>
+    <xacro:property name="wheel_kd" value="100.0"/>
+    <xacro:property name="wheel_mu1" value="1.0"/>
+    <xacro:property name="wheel_mu2" value="1.0"/>
     <!-- The robot is a cylinder 50 cm in diameter and 30 cm in height -->
     <xacro:property name="base_cylinder_radius" value="0.25"/>
@@ -131,4 +135,8 @@
         <gazebo reference="${current_wheel_name}">
             <material>Gazebo/Black</material>
+            <kp>${wheel_kp}</kp>
+            <kd>${wheel_kd}</kd>
+            <mu1>${wheel_mu1}</mu1>
+            <mu2>${wheel_mu2}</mu2>
         </gazebo>
         <joint name="${current_wheel_name}_base_link_joint" type="continuous">
